Commit message: Coupler links working

File: two_coupler_inspector.urdf (robot description, URDF)
Before this commit: robot test_inductor, 3 links, 2 joints
Links:
- link base_link: geometry collision box size=0.1 0.1 0.1; visual box size=0.1 0.1 0.1
- link coupler1_link: mass 1 -> 0.01; geometry collision box size=0.0 0.0 0.0; visual box size=0.05 0.05 0.05
- link coupler2_link: mass 1 -> 0.01; geometry collision box size=0.0 0.0 0.0; visual box size=0.05 0.05 0.05
Joints:
- joint coupler1_joint: axis (none) -> 0 1 0; limit (none) -> lower=-0.01 upper=0.01; origin xyz=0 0.01 0 -> xyz=0 0.15 0; type fixed -> continuous
- joint coupler2_joint: axis (none) -> 0 1 0; limit (none) -> lower=-0.01 upper=0.01; origin xyz=0 -0.01 0 -> xyz=0 -0.15 0; type fixed -> continuous
