Commit message: first urdf_generator commit

File: curve_inspector.xacro (robot description, xacro)
@@ -13,5 +13,5 @@
 	    <origin rpy="0 0 0" xyz="0 0 0" />
 	    <geometry>
-		<box size="0.05 0.05 0.05" />
+		<cylinder length="0.01" radius="0.02"/>
 	    </geometry>
 	</visual>
@@ -29,5 +29,5 @@
 	    <parent link="coupler${coupler_num}_link"/>
 	    <origin xyz="0 0 0"/>
-	    <axis xyz="${axis}"/>
+	    <axis xyz="1 0 0"/><!--make coupler always aligned with x axis of parent link-->
 	</induction_coupler>
     </force_element>

File: two_coupler_inspector.urdf (robot description, URDF)
Before this commit: robot test_inductor, 3 links, 2 joints
Links:
- link coupler1_link: geometry collision box size=0.0 0.0 0.0; visual cylinder length=0.01 radius=0.02
- link coupler2_link: geometry collision box size=0.0 0.0 0.0; visual cylinder length=0.01 radius=0.02
Joints:
- joint coupler2_joint: axis 0 1 0 -> 0 -1 0
